File: ilosuno.kicad_sch (KiCad schematic)
At the start: 44 parts, among them J1 UNPOPULATED_2.54MM_PADS, J2 KF350, J3 UNPOPULATED_2.54MM_PADS, J4 KF350, Q1 IRLR7843TRPBF, Q2 AO3400A, Q3 AO3400A, Q4 IRLR7843TRPBF, Q5 AO3400A, Q6 IRLR7843TRPBF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

Commit message: rev1a: Fixed buck converter output overvoltage bug. Added reverse polarity protection. Exposed more pins to GPIO header (RST, IO2 and IO15)
Parts:
- added D3: SS54/SMA, Diode_SMD:D_SMA, symbol Diode:B340
- added R20: 10k, Resistor_SMD:R_0603_1608Metric, symbol Device:R
- J1: value UNPOPULATED_2.54MM_PADS -> 2.54MM_PADS
- J3: value UNPOPULATED_2.54MM_PADS -> 2.54MM_PADS; footprint Connector_PinHeader_2.54mm:PinHeader_1x05_P2.54mm_Vertical -> Connector_PinHeader_2.54mm:PinHeader_2x05_P2.54mm_Vertical; symbol Connector:Conn_01x05_Socket -> Connector_Generic:Conn_02x05_Odd_Even
- L1: value 68uH/SWPA5040S680MT -> 100uH/SWPA5040S101MT; LCSC C86662 -> C88132
- R18: value 5.6k -> 6k49; JLC Basic Part Y -> N; LCSC C23189 -> C23088
Connections:
- net +3V3: now also J3.3 (Pin_3), J3.4 (Pin_4), R20.1; no longer J3.2 (Pin_2)
- net GND: now also J3.2 (Pin_2)
- net IO16: now also J3.6 (Pin_6); no longer J3.3 (Pin_3)
- net IO5: now also J3.9 (Pin_9); no longer J3.5 (Pin_5)
- net VDD: now also D3.2 (A); no longer C5.1, C8.1, R7.1, U3.7 (VIN)
- net IO15: now reaches R2.1, U1.6 (IO15)
- net IO15: now also J3.8 (Pin_8)
- net RST: now reaches U1.15 (RST)
- net RST: now also J3.5 (Pin_5)
- net IO2: now reaches U1.7 (IO2)
- net IO2: now also J3.10 (Pin_10), R20.2
- net IO6 renamed TOUT
- net TOUT: now also J3.7 (Pin_7); no longer J3.4 (Pin_4)
- new net: C5.1, C8.1, D3.1 (K), R7.1, U3.7 (VIN)
- no-connect marks 2 -> 0
Other:
- note added: "GPIO PORT"
- note added: "NodeMCU D4"
- note added: "NodeMCU D8"
- note added: "Normal boot: IO15 pull down IO2 pull up or left open IO0 pull up or left open To program: PC UART DONGLE <-> DEVICE RTS <-> CH_PD RX <-> ESP_TX TX <-> ESP_RX DTR <-> IO0 3V3 <-> +3V3 (or use external PSU) GND <-> GND"
- note added: "Set point: 3.1V OVP: 3.1*1.125 = 3.49V"
- note removed: "Normal boot: IO15 pull down IO2 pull up or left open IO0 pull high or left open To program: PC UART DONGLE <-> DEVICE RTS <-> CH_PD RX <-> ESP_TX TX <-> ESP_RX DTR <-> IO0 3V3 <-> +3V3 (or use external PSU) GND <-> GND"
- moved on the sheet: C4, C5, C6, C7, C8, D2, J1, J2, L1, R16, R17, R18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
